File: KiCad/_saved_plus_minus_5voltSource.sch (KiCad schematic (older format))
At the start: 16 parts, among them J1 USB_OTG, P1 CONN_01X03, SW1 SW_Push, U1 LM7805_TO220, U2 7660, U3 LM79L05_TO92

Commit message: Edited component association to be all through hole components.
Parts:
- C1, C2: footprint Capacitors_ThroughHole:C_Radial_D5_L6_P2.5 -> Capacitors_ThroughHole:CP_Radial_D5.0mm_P2.50mm
- P1: footprint Pin_Headers:Pin_Header_Angled_1x03 -> Pin_Headers:Pin_Header_Angled_1x03_Pitch2.54mm
Changed lines of the file:
@@
 F 0 "C1" H 5175 3500 50  0000 L CNN
 F 1 "CP" H 5175 3300 50  0000 L CNN
-F 2 "Capacitors_ThroughHole:C_Radial_D5_L6_P2.5" H 5188 3250 30  0001 C CNN
+F 2 "Capacitors_ThroughHole:CP_Radial_D5.0mm_P2.50mm" H 5188 3250 30  0001 C CNN
 F 3 "" H 5150 3400 60  0000 C CNN
 	1    5150 3400
@@
 F 0 "C2" H 6825 3750 50  0000 L CNN
 F 1 "CP" H 6825 3550 50  0000 L CNN
-F 2 "Capacitors_ThroughHole:C_Radial_D5_L6_P2.5" H 6838 3500 30  0001 C CNN
+F 2 "Capacitors_ThroughHole:CP_Radial_D5.0mm_P2.50mm" H 6838 3500 30  0001 C CNN
 F 3 "" H 6800 3650 60  0000 C CNN
 	1    6800 3650
@@
 F 0 "P1" H 6250 4950 50  0000 C CNN
 F 1 "CONN_01X03" V 6350 4750 50  0000 C CNN
-F 2 "Pin_Headers:Pin_Header_Angled_1x03" H 6250 4750 60  0001 C CNN
+F 2 "Pin_Headers:Pin_Header_Angled_1x03_Pitch2.54mm" H 6250 4750 60  0001 C CNN
 F 3 "" H 6250 4750 60  0000 C CNN
 	1    6250 4750

Commit message: Edited BoM to have updated part numbers
Parts:
- D1, D2: footprint LEDs:LED_0805 -> LEDs:LED_D3.0mm
- R1, R2: footprint Resistors_SMD:R_0805_HandSoldering -> Resistors_ThroughHole:R_Axial_DIN0204_L3.6mm_D1.6mm_P5.08mm_Vertical
Changed lines of the file:
@@
 F 0 "D1" H 3150 3650 50  0000 C CNN
 F 1 "LED" H 3150 3450 50  0000 C CNN
-F 2 "LEDs:LED_0805" H 3150 3550 60  0001 C CNN
+F 2 "LEDs:LED_D3.0mm" H 3150 3550 60  0001 C CNN
 F 3 "" H 3150 3550 60  0000 C CNN
 	1    3150 3550
@@
 F 0 "R1" V 3230 3100 50  0000 C CNN
 F 1 "1k" V 3150 3100 50  0000 C CNN
-F 2 "Resistors_SMD:R_0805_HandSoldering" V 3080 3100 30  0001 C CNN
+F 2 "Resistors_ThroughHole:R_Axial_DIN0204_L3.6mm_D1.6mm_P5.08mm_Vertical" V 3080 3100 30  0001 C CNN
 F 3 "" H 3150 3100 30  0000 C CNN
 	1    3150 3100
@@
 F 0 "R2" V 7580 3100 50  0000 C CNN
 F 1 "1k" V 7500 3100 50  0000 C CNN
-F 2 "Resistors_SMD:R_0805_HandSoldering" V 7430 3100 30  0001 C CNN
+F 2 "Resistors_ThroughHole:R_Axial_DIN0204_L3.6mm_D1.6mm_P5.08mm_Vertical" V 7430 3100 30  0001 C CNN
 F 3 "" H 7500 3100 30  0000 C CNN
 	1    7500 3100
@@
 F 0 "D2" H 7500 3650 50  0000 C CNN
 F 1 "LED" H 7500 3450 50  0000 C CNN
-F 2 "LEDs:LED_0805" H 7500 3550 60  0001 C CNN
+F 2 "LEDs:LED_D3.0mm" H 7500 3550 60  0001 C CNN
 F 3 "" H 7500 3550 60  0000 C CNN
 	1    7500 3550
